Commit message: chore: snapshot current simulation updates on temp branch

File: catkin_ws/src/p3at_lms_description/urdf/p3at_lms.urdf.xacro (robot description, xacro)
@@ -1,7 +1,11 @@
 <?xml version="1.0"?>
 <!--
-  P3-AT robot with SICK LMS200 lidar.
-  Uses official Pioneer 3-AT mesh files from amr-ros-config for accurate visual geometry.
-  Adds base_footprint frame, LMS200 lidar link, and Gazebo simulation plugins.
+  P3-AT integrated full-assembly robot model.
+  Includes:
+    - Base chassis/wheels + drive plugin
+    - RPLIDAR A2M12 (rear-underbody, inverted)
+    - Unitree L1 lidar (front-top)
+    - RGBD camera + aluminium strut mount structure
+  Uses official Pioneer 3-AT mesh files for accurate visual geometry.
 -->
 <robot name="p3at_lms" xmlns:xacro="http://www.ros.org/wiki/xacro">
@@ -324,37 +328,155 @@
   <xacro:p3at_drive_side side="left"  reflect="1"/>
   <xacro:p3at_drive_side side="right" reflect="-1"/>
-  <!-- ======================== SICK LMS200 Lidar ======================== -->
+  <!-- ======================== RPLIDAR A2M12 (rear-underbody, inverted) ======================== -->
   <!--
-    Mounted on top plate. The LMS200 is ~0.185m tall, sits on the top plate at z=0.274.
-    laser frame origin at the scanner emission plane.
+    User mounting requirement (real robot):
+      - Mounted under the rear of the chassis ("车屁股下面")
+      - Laterally centered (y=0)
+      - 1 cm inward from rear outer edge
+      - Sensor installed upside-down
+    Coordinate convention used here:
+      - base_link: +x forward, +y left, +z up
+      - P3AT chassis projection rear edge from collision box: x=-0.25 m
+      - A2 outer radius approximated as 0.038 m
+      - required outer rear edge target: -0.25 + 0.01 = -0.24 m
+      - baseline center x from geometry: -0.24 + 0.038 = -0.202 m
+      - calibrated runtime offset: x = -0.232 m (shifted further rear by 3 cm)
+      - chassis lower surface approximated from base collision box bottom: z=0.097 m
+      - A2M12 body height approximated as 0.05 m (visual/collision)
+    To satisfy "lidar lower face bonded to chassis lower face" with inverted mount,
+    place laser joint at z=0.072 m and rotate 180 deg around X.
   -->
   <link name="laser">
     <inertial>
-      <mass value="4.5"/>
-      <origin xyz="0 0 0"/>
-      <inertia ixx="0.01" ixy="0.0" ixz="0.0"
-               iyy="0.01" iyz="0.0"
-               izz="0.01"/>
-    </inertial>
-    <visual>
-      <origin xyz="0 0 0" rpy="0 0 0"/>
-      <geometry>
-        <box size="0.156 0.155 0.185"/>
-      </geometry>
-      <material name="LMS200Blue">
-        <color rgba="0.12 0.34 0.56 1.0"/>
-      </material>
-    </visual>
-    <!-- No collision: prevents Gazebo ray sensor self-collision
-         after fixed-joint link merging into base_link -->
-  </link>
-  <gazebo reference="laser">
-    <material>Gazebo/Blue</material>
-  </gazebo>
+      <mass value="0.19"/>
+      <origin xyz="0 0 0"/>
+      <inertia ixx="0.0003" ixy="0.0" ixz="0.0"
+               iyy="0.0003" iyz="0.0"
+               izz="0.0003"/>
+    </inertial>
+    <visual>
+      <origin xyz="0 0 0" rpy="0 0 0"/>
+      <geometry>
+        <!-- Approximate A2 body (diameter ~76mm, height ~50mm) -->
+        <cylinder radius="0.038" length="0.05"/>
+      </geometry>
+      <material name="RplidarGrey">
+        <color rgba="0.25 0.25 0.25 1.0"/>
+      </material>
+    </visual>
+    <collision>
+      <origin xyz="0 0 0" rpy="0 0 0"/>
+      <geometry>
+        <cylinder radius="0.038" length="0.05"/>
+      </geometry>
+    </collision>
+    <!-- Collision kept for RViz/URDF inspection; Gazebo ray tracing still uses sensor plugin -->
+  </link>
+  <gazebo reference="laser"><material>Gazebo/DarkGrey</material></gazebo>
   <joint name="laser_joint" type="fixed">
     <parent link="base_link"/>
     <child link="laser"/>
-    <!-- On top plate center, raised to emission plane -->
-    <origin xyz="0.0 0.0 0.366" rpy="0 0 0"/>
+    <!-- Rear-underbody, centered, upside-down; outer rim is 1cm inside rear edge -->
+    <origin xyz="-0.232 0.0 0.072" rpy="3.1415926535897931 0 0"/>
+  </joint>
+  <!-- ======================== Unitree 4D Lidar L1 (front-top) ======================== -->
+  <!--
+    Keep Unitree frame definition in the same full robot URDF for visualization/
+    calibration checks. Runtime can still choose which LiDAR topic to consume.
+  -->
+  <xacro:include filename="$(find p3at_lms_description)/urdf/unitree_lidar_l1.urdf.xacro"/>
+  <xacro:unitree_lidar_l1 parent="base_link" prefix="unitree"
+                           xyz="0.208 0.0 0.299" rpy="0 0 0"
+                           sim_scan_topic="unitree/scan"
+                           sim_cloud_topic="unitree/cloud"
+                           sim_imu_topic="unitree/imu"
+                           enable_3d="true"/>
+  <!-- ======================== Aluminium Struts + RGBD Camera ======================== -->
+  <!--
+    Camera mount follows existing deployment convention:
+      - camera center at x=0.208, y=0, z=0.85
+      - camera optical orientation remains managed by launch-time static TF
+    Two aluminum struts are modeled as vertical cylindrical links.
+    Strut lower end touches top plate upper surface at z=0.274.
+  -->
+  <link name="left_aluminum_strut">
+    <inertial>
+      <mass value="0.25"/>
+      <origin xyz="0 0 0"/>
+      <inertia ixx="0.0008" ixy="0" ixz="0" iyy="0.0008" iyz="0" izz="0.00005"/>
+    </inertial>
+    <visual>
+      <origin xyz="0 0 0" rpy="0 0 0"/>
+      <geometry>
+        <cylinder radius="0.01" length="0.70"/>
+      </geometry>
+      <material name="AluminiumSilver">
+        <color rgba="0.72 0.74 0.76 1.0"/>
+      </material>
+    </visual>
+  </link>
+  <joint name="left_aluminum_strut_joint" type="fixed">
+    <parent link="base_link"/>
+    <child link="left_aluminum_strut"/>
+    <origin xyz="0.18 0.08 0.624" rpy="0 0 0"/>
+  </joint>
+  <link name="right_aluminum_strut">
+    <inertial>
+      <mass value="0.25"/>
+      <origin xyz="0 0 0"/>
+      <inertia ixx="0.0008" ixy="0" ixz="0" iyy="0.0008" iyz="0" izz="0.00005"/>
+    </inertial>
+    <visual>
+      <origin xyz="0 0 0" rpy="0 0 0"/>
+      <geometry>
+        <cylinder radius="0.01" length="0.70"/>
+      </geometry>
+      <material name="AluminiumSilver"/>
+    </visual>
+  </link>
+  <joint name="right_aluminum_strut_joint" type="fixed">
+    <parent link="base_link"/>
+    <child link="right_aluminum_strut"/>
+    <origin xyz="0.18 -0.08 0.624" rpy="0 0 0"/>
+  </joint>
+  <link name="rgbd_camera_mount_bar">
+    <inertial>
+      <mass value="0.12"/>
+      <origin xyz="0 0 0"/>
+      <inertia ixx="0.0002" ixy="0" ixz="0" iyy="0.00002" iyz="0" izz="0.0002"/>
+    </inertial>
+    <visual>
+      <origin xyz="0 0 0" rpy="0 0 0"/>
+      <geometry>
+        <box size="0.02 0.18 0.02"/>
+      </geometry>
+      <material name="AluminiumSilver"/>
+    </visual>
+  </link>
+  <joint name="rgbd_camera_mount_bar_joint" type="fixed">
+    <parent link="base_link"/>
+    <child link="rgbd_camera_mount_bar"/>
+    <origin xyz="0.208 0.0 0.85" rpy="0 0 0"/>
+  </joint>
+  <link name="rgbd_camera">
+    <inertial>
+      <mass value="0.09"/>
+      <origin xyz="0 0 0"/>
+      <inertia ixx="0.00005" ixy="0" ixz="0" iyy="0.00005" iyz="0" izz="0.00002"/>
+    </inertial>
+    <visual>
+      <origin xyz="0.0 0.0 0.0" rpy="0 0 0"/>
+      <geometry>
+        <box size="0.09 0.025 0.025"/>
+      </geometry>
+      <material name="CameraBlack">
+        <color rgba="0.08 0.08 0.08 1.0"/>
+      </material>
+    </visual>
+  </link>
+  <joint name="rgbd_camera_joint" type="fixed">
+    <parent link="rgbd_camera_mount_bar"/>
+    <child link="rgbd_camera"/>
+    <origin xyz="0.0 0.0 0.0" rpy="0 0 0"/>
   </joint>
   <!-- ======================== Gazebo Skid-Steer Drive Plugin ======================== -->
@@ -380,7 +502,7 @@
     </plugin>
   </gazebo>
-  <!-- ======================== Gazebo LMS200 Lidar Sensor ======================== -->
+  <!-- ======================== Gazebo RPLIDAR-like 2D Sensor ======================== -->
   <gazebo reference="laser">
-    <sensor type="ray" name="lms200">
+    <sensor type="ray" name="rplidar_a2m12">
       <pose>0 0 0 0 0 0</pose>
       <visualize>true</visualize>
@@ -389,13 +511,13 @@
         <scan>
           <horizontal>
-            <samples>361</samples>
+            <samples>720</samples>
             <resolution>1</resolution>
-            <min_angle>-1.57079632679</min_angle>
-            <max_angle> 1.57079632679</max_angle>
+            <min_angle>-3.1415926535897931</min_angle>
+            <max_angle> 3.1415926535897931</max_angle>
           </horizontal>
         </scan>
         <range>
-          <min>0.05</min>
-          <max>30.0</max>
+          <min>0.2</min>
+          <max>12.0</max>
           <resolution>0.01</resolution>
         </range>
