Commit message: main: migrate to URDF-authoritative sensor extrinsics and add full sim regression evidence
This commit consolidates the real-deployment navigation/target-follow stack
around a single authoritative extrinsics source (p3at_unitree.urdf.xacro),
fixes follower stability issues found in simulation retest, aligns script
entrypoints with the migrated launch chain, and archives full regression logs.

What was changed

1) URDF/TF authority migration (single source of truth)
- Updated p3at_unitree URDF to explicitly carry the dual-lidar + camera layout:
  - RPLIDAR frame `laser` fixed joint at x=-0.272, y=0.0, z=0.072, inverted mount.
  - RGBD mounting link + `camera_link` optical frame using optical convention.
- Kept file name unchanged as requested:
  - catkin_ws/src/p3at_lms_description/urdf/p3at_unitree.urdf.xacro

2) Real-robot launch chain alignment to URDF-authoritative TF
- Removed legacy duplicate static TF assumptions from real launch path.
- Ensured launch chain uses robot_state_publisher/URDF extrinsics consistently.
- Updated these launch files:
  - catkin_ws/src/p3at_lms_navigation/launch/real_robot_lidar_bringup.launch
  - catkin_ws/src/p3at_lms_navigation/launch/real_robot_mapping_unitree.launch
  - catkin_ws/src/p3at_lms_navigation/launch/real_robot_mapping_rplidar.launch
  - catkin_ws/src/p3at_lms_navigation/launch/real_robot_nav_unitree.launch
  - catkin_ws/src/p3at_lms_navigation/launch/real_robot_nav_rplidar.launch
  - catkin_ws/src/target_follower/launch/target_follow_real.launch

3) Target follower robustness fixes (core runtime logic)
- Fixed startup crash in sim-time windows:
  - guarded path/dialogue memory cutoff computations against negative time.
- Improved exploration scan gating diagnostics and behavior:
  - `_can_scan_in_place()` now returns reason codes,
  - avoids false hard-block from costmap startup edge cases,
  - emits clearer skip reasons in logs.
- File:
  - catkin_ws/src/target_follower/scripts/target_follower.py

4) Script entrypoint migration (real operation path)
- Updated scripts/start_demo.sh to match migrated launch API and URDF authority:
  - removed deprecated `camera_tf_*` / `rplidar_tf_*` passthrough args,
  - removed stale “approx TF” warning path tied to old static TF flow,
  - fixed overlay target-follow launch to explicitly pass `global_frame:=map`.

5) Launch arg stability hardening
- Set target_follow_real.launch `global_frame` default to `map` so
  overlay mode does not fail when caller omits `global_frame`.

6) Full simulation retest artifacts committed
- Added reproducible retest scripts and complete logs/metrics under:
  - Log/sim_retest_20260318/
  - including iterative v2/v3/v4 scripts and per-run outputs.

Key verified outcomes from latest passing run
- Artifact:
  Log/sim_retest_20260318/20260318_085328_v3/metrics/full_logic_retest_summary_v3.json
- `overall_pass: true`
- Auto-explore entered and ran (`auto_explore_ok: true`)
- Case A (action=false) path observed through WAITING_ACTION -> RETREATING
- Case B (action=true) path observed through WAITING_ACTION -> POST_ACCEPT_COOLDOWN -> RETREATING
- TF checks matched migrated URDF authority:
  - base_link -> laser      = (-0.272, 0.0, 0.072)
  - base_link -> camera_link = (0.208, 0.0, 0.85)
- No non-shutdown traceback flagged in final summary (`traceback_found: false`)

Notes
- This commit intentionally includes full raw experiment/retest logs for
  traceability and paper/report reproducibility.

File: catkin_ws/src/p3at_lms_description/urdf/p3at_unitree.urdf.xacro (robot description, xacro)
@@ -1,10 +1,6 @@
 <?xml version="1.0"?>
 <!--
-  P3-AT robot with Unitree 4D Lidar L1 ONLY (SICK LMS200 removed).
-  - Full P3-AT chassis, wheels, and drive plugin
-  - Unitree 4D Lidar L1 mounted at z=0.366 (same position as former SICK)
-    - 2D LaserScan: /unitree/scan  (frame: unitree_lidar)  360° FOV
-    - 3D PointCloud2: /unitree/cloud (frame: unitree_lidar)
-    - IMU: /unitree/imu (frame: unitree_imu)
+  P3-AT robot with Unitree + RPLIDAR + RGBD camera extrinsics.
+  This file is the single source of truth for base_link sensor extrinsics.
 -->
 <robot name="p3at_unitree" xmlns:xacro="http://www.ros.org/wiki/xacro">
@@ -318,4 +314,79 @@
   <xacro:p3at_drive_side side="left"  reflect="1"/>
   <xacro:p3at_drive_side side="right" reflect="-1"/>
+  <!-- ======================== RPLIDAR A2M12 (rear-underbody, inverted) ======================== -->
+  <!--
+    Mounting requirement:
+      - Rear-underbody, centered at y=0
+      - x is fixed to -0.272 m (latest calibrated value)
+      - z=0.072 m
+      - Sensor mounted upside-down (roll = pi)
+  -->
+  <link name="laser">
+    <inertial>
+      <mass value="0.19"/>
+      <origin xyz="0 0 0"/>
+      <inertia ixx="0.0003" ixy="0.0" ixz="0.0"
+               iyy="0.0003" iyz="0.0"
+               izz="0.0003"/>
+    </inertial>
+    <visual>
+      <origin xyz="0 0 0" rpy="0 0 0"/>
+      <geometry>
+        <cylinder radius="0.038" length="0.05"/>
+      </geometry>
+      <material name="RplidarGrey">
+        <color rgba="0.25 0.25 0.25 1.0"/>
+      </material>
+    </visual>
+    <collision>
+      <origin xyz="0 0 0" rpy="0 0 0"/>
+      <geometry>
+        <cylinder radius="0.038" length="0.05"/>
+      </geometry>
+    </collision>
+  </link>
+  <gazebo reference="laser">
+    <material>Gazebo/DarkGrey</material>
+  </gazebo>
+  <joint name="laser_joint" type="fixed">
+    <parent link="base_link"/>
+    <child link="laser"/>
+    <origin xyz="-0.272 0.0 0.072" rpy="${PI} 0 0"/>
+  </joint>
+  <!-- ======================== RGBD camera + optical frame ======================== -->
+  <!--
+    camera_link is intentionally defined as the optical frame:
+      x = right, y = down, z = forward
+    so perception outputs in camera_link can be consumed directly.
+  -->
+  <link name="rgbd_camera">
+    <inertial>
+      <mass value="0.09"/>
+      <origin xyz="0 0 0"/>
+      <inertia ixx="0.00005" ixy="0" ixz="0"
+               iyy="0.00005" iyz="0"
+               izz="0.00002"/>
+    </inertial>
+    <visual>
+      <origin xyz="0.0 0.0 0.0" rpy="0 0 0"/>
+      <geometry>
+        <box size="0.09 0.025 0.025"/>
+      </geometry>
+      <material name="CameraBlack">
+        <color rgba="0.08 0.08 0.08 1.0"/>
+      </material>
+    </visual>
+  </link>
+  <joint name="rgbd_camera_joint" type="fixed">
+    <parent link="base_link"/>
+    <child link="rgbd_camera"/>
+    <origin xyz="0.208 0.0 0.85" rpy="0 0 0"/>
+  </joint>
+  <link name="camera_link"/>
+  <joint name="camera_optical_joint" type="fixed">
+    <parent link="rgbd_camera"/>
+    <child link="camera_link"/>
+    <origin xyz="0 0 0" rpy="${-PI/2} 0 ${-PI/2}"/>
+  </joint>
   <!-- ======================== Gazebo Skid-Steer Drive Plugin ======================== -->
   <gazebo>

Commit message: fix problem of yolo kill itself at starting

File: catkin_ws/src/p3at_lms_description/urdf/p3at_unitree.urdf.xacro (robot description, xacro)
@@ -420,10 +420,131 @@
       → 雷达中心 z = 0.274 + 0.025 = 0.299
   -->
-  <xacro:include filename="$(find p3at_lms_description)/urdf/unitree_lidar_l1.urdf.xacro"/>
-  <xacro:unitree_lidar_l1 parent="base_link" prefix="unitree"
-                           xyz="0.208 0.0 0.299" rpy="0 0 0"
-                           sim_scan_topic="unitree/scan"
-                           sim_cloud_topic="unitree/cloud"
-                           sim_imu_topic="unitree/imu"
-                           enable_3d="true"/>
+  <link name="unitree_lidar">
+    <inertial>
+      <mass value="0.05"/>
+      <origin xyz="0 0 0" rpy="0 0 0"/>
+      <inertia ixx="0.00004" ixy="0.0" ixz="0.0"
+               iyy="0.00004" iyz="0.0"
+               izz="0.00004"/>
+    </inertial>
+    <visual>
+      <origin xyz="0 0 0" rpy="0 0 0"/>
+      <geometry>
+        <cylinder radius="0.0325" length="0.050"/>
+      </geometry>
+      <material name="UnitreeLidarBlack">
+        <color rgba="0.15 0.15 0.15 1.0"/>
+      </material>
+    </visual>
+  </link>
+  <gazebo reference="unitree_lidar">
+    <material>Gazebo/DarkGrey</material>
+  </gazebo>
+  <joint name="unitree_lidar_joint" type="fixed">
+    <parent link="base_link"/>
+    <child link="unitree_lidar"/>
+    <origin xyz="0.208 0.0 0.299" rpy="0 0 0"/>
+  </joint>
+  <link name="unitree_imu">
+    <inertial>
+      <mass value="0.001"/>
+      <origin xyz="0 0 0"/>
+      <inertia ixx="0.0001" ixy="0.0" ixz="0.0"
+               iyy="0.0001" iyz="0.0"
+               izz="0.0001"/>
+    </inertial>
+  </link>
+  <joint name="unitree_imu_joint" type="fixed">
+    <parent link="unitree_lidar"/>
+    <child link="unitree_imu"/>
+    <origin xyz="0 0 0" rpy="0 0 0"/>
+  </joint>
+  <gazebo reference="unitree_lidar">
+    <sensor type="ray" name="unitree_lidar_2d">
+      <pose>0 0 0 0 0 0</pose>
+      <visualize>true</visualize>
+      <update_rate>15</update_rate>
+      <ray>
+        <scan>
+          <horizontal>
+            <samples>720</samples>
+            <resolution>1</resolution>
+            <min_angle>-${PI}</min_angle>
+            <max_angle>${PI}</max_angle>
+          </horizontal>
+        </scan>
+        <range>
+          <min>0.05</min>
+          <max>30.0</max>
+          <resolution>0.01</resolution>
+        </range>
+        <noise>
+          <type>gaussian</type>
+          <mean>0.0</mean>
+          <stddev>0.005</stddev>
+        </noise>
+      </ray>
+      <plugin name="gazebo_ros_unitree_laser" filename="libgazebo_ros_laser.so">
+        <topicName>unitree/scan</topicName>
+        <frameName>unitree_lidar</frameName>
+      </plugin>
+    </sensor>
+  </gazebo>
+  <gazebo reference="unitree_lidar">
+    <sensor type="ray" name="unitree_lidar_3d">
+      <pose>0 0 0 0 0 0</pose>
+      <visualize>false</visualize>
+      <update_rate>10</update_rate>
+      <ray>
+        <scan>
+          <horizontal>
+            <samples>360</samples>
+            <resolution>1</resolution>
+            <min_angle>-${PI}</min_angle>
+            <max_angle>${PI}</max_angle>
+          </horizontal>
+          <vertical>
+            <samples>16</samples>
+            <resolution>1</resolution>
+            <min_angle>-${15*PI/180}</min_angle>
+            <max_angle>${52*PI/180}</max_angle>
+          </vertical>
+        </scan>
+        <range>
+          <min>0.05</min>
+          <max>30.0</max>
+          <resolution>0.02</resolution>
+        </range>
+        <noise>
+          <type>gaussian</type>
+          <mean>0.0</mean>
+          <stddev>0.008</stddev>
+        </noise>
+      </ray>
+      <plugin name="gazebo_ros_unitree_cloud" filename="libgazebo_ros_block_laser.so">
+        <topicName>unitree/cloud</topicName>
+        <frameName>unitree_lidar</frameName>
+        <updateRate>10.0</updateRate>
+      </plugin>
+    </sensor>
+  </gazebo>
+  <gazebo reference="unitree_imu">
+    <gravity>true</gravity>
+    <sensor name="unitree_imu_sensor" type="imu">
+      <always_on>true</always_on>
+      <update_rate>200</update_rate>
+      <visualize>false</visualize>
+      <topic>unitree/imu</topic>
+      <plugin filename="libgazebo_ros_imu_sensor.so" name="unitree_imu_plugin">
+        <topicName>unitree/imu</topicName>
+        <bodyName>unitree_imu</bodyName>
+        <updateRateHZ>200.0</updateRateHZ>
+        <gaussianNoise>0.0</gaussianNoise>
+        <xyzOffset>0 0 0</xyzOffset>
+        <rpyOffset>0 0 0</rpyOffset>
+        <frameName>unitree_imu</frameName>
+      </plugin>
+      <pose>0 0 0 0 0 0</pose>
+    </sensor>
+  </gazebo>
 </robot>
